File: Dev board 1/KiCAD/UKDAQ/UKDAQ.kicad_sch (KiCad schematic)
At the start: 22 parts, among them J1 5 pin Molex (0537800570), U1 AP2210N_SOT-23-3, U2 PI4ULS5V202, U3 BNO055, U4 BME280, U5 MAX32660-24TQFN-EP, Y1 Crystal

Commit message: updated dev board 1 to rev 2 design
Parts:
- removed U5: MAX32660-24TQFN-EP, Joseph:MAX32660-24-TQFN-EP, symbol Joseph:MAX32660-24TQFN-EP
- added J2: Conn_01x11_Male, Connector_PinHeader_2.54mm:PinHeader_1x11_P2.54mm_Vertical, symbol Connector:Conn_01x11_Male
- added U5: MAX32660-20TQFN-EP, Package_DFN_QFN:QFN-20-1EP_5x5mm_P0.65mm_EP3.35x3.35mm, symbol Joseph:MAX32660-20TQFN-EP
- C1, C2, C9: footprint Capacitor_SMD:C_0201_0603Metric -> Capacitor_SMD:C_0603_1608Metric
- C10: value 1 uF -> 100 nF; footprint Capacitor_SMD:C_0201_0603Metric -> Capacitor_SMD:C_0603_1608Metric
- C5: value 6 pF -> 1 uF; footprint Capacitor_SMD:C_01005_0402Metric -> Capacitor_SMD:C_0603_1608Metric
- C6: value 100 nF -> 6 pF
- C8: footprint Capacitor_SMD:C_01005_0402Metric -> Capacitor_SMD:C_0603_1608Metric
- R1: value 10k -> 4.7k
- R2: value 10 -> 4.7k; footprint Resistor_SMD:R_0201_0603Metric -> Resistor_SMD:R_0402_1005Metric
- R4: value 4.7k -> 10k
- R5: value 4.7k -> 10
- U2: footprint Package_DFN_QFN:OnSemi_UDFN-8_1.2x1.8mm_P0.4mm -> Joseph:MSOP-8
Connections:
- net BNO_INTERRUPT: now also J2.8 (Pin_8), U5.13 (P0.11/SPI1_MOSI/UART1_RX)
- net GND: now also C6.2, R5.2, J2.11 (Pin_11), U5.- (EP), U5.6 (VSS); no longer C10.2, R2.2
- net RX/SWCLK-VCC: now also J2.3 (Pin_3)
- net RX/SWCLK-VDD: now also J2.1 (Pin_1), U5.1 (P0.1/SWDCLK/SPI1_MOSI/UART1_RX)
- net SCL: now also R1.2, J2.6 (Pin_6), U5.20 (P0.2/I2C1_SCL/SPI1_SCK/32KCAL); no longer R4.2
- net SDA: now also R2.2, J2.5 (Pin_5), U5.19 (P0.3/I2C1_SDA/SPI1_SSO/TMR0); no longer R5.2
- net TX/SWDIO-VCC: now also J2.4 (Pin_4)
- net TX/SWDIO-VDD: now also J2.2 (Pin_2), U5.2 (P0.0/SWDIO/SPI1_MISO/UART1_TX)
- net VCC: now also J2.10 (Pin_10)
- net VDD: now also R2.1, J2.9 (Pin_9), U5.9 (VDD); no longer R5.1
- net nRESET: now also C10.1, R4.2, J2.7 (Pin_7), U5.5 (RSTN); no longer C6.1, R1.2
- net at C8.1, Y1.1: now also U5.8 (32KIN)
- net at C5.1: now also U5.10 (VCORE); no longer Y1.2
- new net: C10.2, R5.1
- new net: C6.1, U5.7 (32KOUT), Y1.2
Other:
- note added: "Test Grips"
- moved on the sheet: C4, C7, C9, R3, U3, U4

Commit message: small change to MCU footprint
Parts:
- U5: footprint Package_DFN_QFN:QFN-20-1EP_5x5mm_P0.65mm_EP3.35x3.35mm -> Package_DFN_QFN:TQFN-20-1EP_5x5mm_P0.65mm_EP3.1x3.1mm
Connections:
- net GND: now also U5.21 (EP); no longer U5.- (EP)
Changed lines of the file:
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@@
       (effects (font (size 1.27 1.27)) (justify right))
     )
-    (property "Footprint" "Package_DFN_QFN:QFN-20-1EP_5x5mm_P0.65mm_EP3.35x3.35mm" (id 2) (at 63.5 185.42 0)
+    (property "Footprint" "Package_DFN_QFN:TQFN-20-1EP_5x5mm_P0.65mm_EP3.1x3.1mm" (id 2) (at 63.5 185.42 0)
       (effects (font (size 1.27 1.27)) hide)
     )
@@
       (effects (font (size 1.27 1.27)) hide)
     )
-    (pin "-")
     (pin "1")
     (pin "10")
@@
     (pin "2")
     (pin "20")
+    (pin "21")
     (pin "3")
     (pin "4")
@@
     )
     (path "/ecd46510-660b-4043-b957-ccc94f56b0ca"
-      (reference "U5") (unit 1) (value "MAX32660-20TQFN-EP") (footprint "Package_DFN_QFN:QFN-20-1EP_5x5mm_P0.65mm_EP3.35x3.35mm")
+      (reference "U5") (unit 1) (value "MAX32660-20TQFN-EP") (footprint "Package_DFN_QFN:TQFN-20-1EP_5x5mm_P0.65mm_EP3.1x3.1mm")
     )
     (path "/b83c4dba-2e1b-4066-afd5-e4ee51eb7927"

Commit message: changes to board design and new BOM
Parts:
- U5: footprint Package_DFN_QFN:TQFN-20-1EP_5x5mm_P0.65mm_EP3.1x3.1mm -> Joseph:21-0139V_T2044&plus_5_MXM
Changed lines of the file:
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@@
       (effects (font (size 1.27 1.27)) (justify right))
     )
-    (property "Footprint" "Package_DFN_QFN:TQFN-20-1EP_5x5mm_P0.65mm_EP3.1x3.1mm" (id 2) (at 63.5 185.42 0)
+    (property "Footprint" "Joseph:21-0139V_T2044&plus_5_MXM" (id 2) (at 63.5 185.42 0)
       (effects (font (size 1.27 1.27)) hide)
     )
@@
     )
     (path "/ecd46510-660b-4043-b957-ccc94f56b0ca"
-      (reference "U5") (unit 1) (value "MAX32660-20TQFN-EP") (footprint "Package_DFN_QFN:TQFN-20-1EP_5x5mm_P0.65mm_EP3.1x3.1mm")
+      (reference "U5") (unit 1) (value "MAX32660-20TQFN-EP") (footprint "Joseph:21-0139V_T2044&plus_5_MXM")
     )
     (path "/b83c4dba-2e1b-4066-afd5-e4ee51eb7927"
